File: hardware/HP35_Z80.brd (EAGLE design)
At the start: 235 x 202 mm, 82 parts, among them IC4 74HCT32N, IC5 74HCT154N, IC6 74HCT138N, IC7 74HCT541N, IC8 74HCT573N, IC9 74HCT573N, X1 MINI-USB-32005-301, X2 MINI-USB-32005-301

Commit message: add gerbers
Connections:
- new net CS: IC2.20, IC4.8
- net /MREQ: now also IC4.10
- net A15: now also IC4.9; no longer IC2.20
- net GND: no longer IC4.10, IC4.9
Routing:
- net CS: track 0.00 -> 65.2 mm, vias 0 -> 1
- net A15: track 64.6 -> 82.4 mm
- net /MREQ: track 46.6 -> 52.7 mm
- net GND: track 155.0 -> 155.9 mm
Changed lines of the file:
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@@
 <contactref element="IC4" pad="12"/>
 <contactref element="IC4" pad="13"/>
-<contactref element="IC4" pad="9"/>
-<contactref element="IC4" pad="10"/>
 <contactref element="IC5" pad="12"/>
 <contactref element="IC7" pad="1"/>
@@
 <contactref element="X2" pad="5"/>
 <contactref element="C12" pad="-"/>
-<wire x1="158.29" y1="146.99" x2="155.88" y2="146.99" width="0.508" layer="16"/>
-<wire x1="155.88" y1="146.99" x2="154.94" y2="146.05" width="0.508" layer="16"/>
-<wire x1="-59" y1="150.19" x2="-57.1375" y2="150.19" width="0.508" layer="16"/>
-<wire x1="-57.1375" y1="150.19" x2="-56.515" y2="150.8125" width="0.508" layer="16"/>
 <via x="10.16" y="67.945" extent="1-16" drill="0.6"/>
 <wire x1="10.16" y1="67.945" x2="12.065" y2="67.31" width="1.27" layer="16"/>
 <wire x1="-16.51" y1="71.12" x2="-16.51" y2="67.945" width="1.27" layer="1"/>
+<wire x1="-59" y1="150.19" x2="-57.328" y2="150.19" width="0.6096" layer="16"/>
+<wire x1="-57.328" y1="150.19" x2="-55.372" y2="151.638" width="0.6096" layer="16"/>
+<wire x1="158.29" y1="146.99" x2="156.388" y2="146.99" width="0.6096" layer="16"/>
+<wire x1="156.388" y1="146.99" x2="155.448" y2="146.05" width="0.6096" layer="16"/>
 </signal>
 <signal name="R5">
@@
 <signal name="A15">
 <contactref element="IC1" pad="5"/>
+<contactref element="IC4" pad="9"/>
+<wire x1="-34.29" y1="55.88" x2="-34.29" y2="50.8" width="0.4064" layer="16"/>
+<via x="-34.29" y="50.8" extent="1-16" drill="0.6"/>
+<wire x1="-34.29" y1="50.8" x2="13.716" y2="50.8" width="0.4064" layer="1"/>
+<wire x1="13.716" y1="50.8" x2="13.97" y2="50.546" width="0.4064" layer="1"/>
+<via x="13.97" y="50.546" extent="1-16" drill="0.6"/>
+<wire x1="13.97" y1="50.546" x2="13.97" y2="36.83" width="0.4064" layer="16"/>
 <contactref element="IC3" pad="26"/>
-<contactref element="IC2" pad="20"/>
-<wire x1="-24.13" y1="12.7" x2="-24.13" y2="19.05" width="0.4064" layer="16"/>
-<wire x1="-24.13" y1="19.05" x2="-25.4" y2="20.32" width="0.4064" layer="16"/>
-<wire x1="-25.4" y1="20.32" x2="-25.4" y2="31.75" width="0.4064" layer="16"/>
-<wire x1="-25.4" y1="31.75" x2="-24.13" y2="33.02" width="0.4064" layer="16"/>
-<wire x1="-24.13" y1="33.02" x2="-24.13" y2="34.29" width="0.4064" layer="16"/>
-<via x="-24.13" y="34.29" extent="1-16" drill="0.6"/>
-<wire x1="-24.13" y1="34.29" x2="-39.37" y2="34.29" width="0.4064" layer="1"/>
-<via x="-39.37" y="34.29" extent="1-16" drill="0.6"/>
-<wire x1="-39.37" y1="34.29" x2="-39.37" y2="40.64" width="0.4064" layer="16"/>
 <wire x1="-39.37" y1="40.64" x2="-39.37" y2="46.99" width="0.4064" layer="16"/>
 <via x="-39.37" y="46.99" extent="1-16" drill="0.6"/>
 <wire x1="-39.37" y1="46.99" x2="-34.29" y2="46.99" width="0.4064" layer="1"/>
 <via x="-34.29" y="46.99" extent="1-16" drill="0.6"/>
-<wire x1="-34.29" y1="46.99" x2="-34.29" y2="55.88" width="0.4064" layer="16"/>
+<wire x1="-34.29" y1="46.99" x2="-34.29" y2="50.8" width="0.4064" layer="16"/>
 </signal>
 <signal name="N$31">
@@
 <wire x1="1.27" y1="55.88" x2="1.27" y2="46.99" width="0.4064" layer="16"/>
 <wire x1="1.27" y1="46.99" x2="-3.81" y2="41.91" width="0.4064" layer="16"/>
-<wire x1="-3.81" y1="41.91" x2="-3.81" y2="30.48" width="0.4064" layer="16"/>
+<wire x1="-3.81" y1="41.91" x2="-3.81" y2="29.21" width="0.4064" layer="16"/>
 <wire x1="1.27" y1="29.21" x2="1.27" y2="31.75" width="0.4064" layer="16"/>
 <wire x1="1.27" y1="31.75" x2="8.89" y2="31.75" width="0.4064" layer="16"/>
@@
 <wire x1="1.27" y1="29.21" x2="-3.81" y2="29.21" width="0.4064" layer="1"/>
 <via x="-3.81" y="29.21" extent="1-16" drill="0.6"/>
-<wire x1="-3.81" y1="29.21" x2="-3.81" y2="30.48" width="0.4064" layer="16"/>
+<contactref element="IC4" pad="10"/>
+<wire x1="11.43" y1="36.83" x2="11.43" y2="34.29" width="0.4064" layer="16"/>
+<wire x1="11.43" y1="34.29" x2="8.89" y2="31.75" width="0.4064" layer="16"/>
 </signal>
 <signal name="/IORQ">
@@
 <wire x1="134.35" y1="154.67" x2="134.35" y2="157.38" width="0.4064" layer="1"/>
 </signal>
+<signal name="CS">
+<contactref element="IC4" pad="8"/>
+<contactref element="IC2" pad="20"/>
+<via x="-24.13" y="34.29" extent="1-16" drill="0.6"/>
+<wire x1="-24.13" y1="34.29" x2="-24.13" y2="33.02" width="0.4064" layer="16"/>
+<wire x1="-24.13" y1="33.02" x2="-25.4" y2="31.75" width="0.4064" layer="16"/>
+<wire x1="-25.4" y1="31.75" x2="-25.4" y2="20.32" width="0.4064" layer="16"/>
+<wire x1="-25.4" y1="20.32" x2="-24.13" y2="19.05" width="0.4064" layer="16"/>
+<wire x1="-24.13" y1="19.05" x2="-24.13" y2="12.7" width="0.4064" layer="16"/>
+<wire x1="16.51" y1="36.83" x2="16.51" y2="35.306" width="0.4064" layer="1"/>
+<wire x1="16.51" y1="35.306" x2="15.494" y2="34.29" width="0.4064" layer="1"/>
+<wire x1="15.494" y1="34.29" x2="-24.13" y2="34.29" width="0.4064" layer="1"/>
+</signal>
+<signal name="N$7">
+</signal>
 </signals>

Commit message: update pcb
Parts:
- added R10, R11, R12, R13, R14, R15, R16, R17: (no value), rcl:R1206
Connections:
- removed net N$35: DIS1.P$11, DIS2.P$11, DIS3.P$11, DIS4.P$11, IC9.19
- new net N$10: IC9.13, R16.1
- new net N$11: IC9.14, R15.1
- new net N$12: IC9.15, R14.1
- new net N$24: IC9.16, R13.1
- new net N$25: IC9.17, R12.1
- new net N$26: IC9.18, R11.1
- new net N$27: IC9.19, R10.1
- new net N$28: DIS1.P$11, DIS2.P$11, DIS3.P$11, DIS4.P$11, R10.2
- new net N$9: IC9.12, R17.1
- net N$31: now also R17.2; no longer IC9.12
- net N$32: now also R16.2; no longer IC9.13
- net N$33: now also R15.2; no longer IC9.14
- net N$34: now also R14.2; no longer IC9.15
- net N$36: now also R11.2; no longer IC9.18
- net N$37: now also R12.2; no longer IC9.17
- net N$38: now also R13.2; no longer IC9.16
Routing:
- net N$35: track 222.5 -> 0.00 mm, vias 5 -> 0
- net N$28: track 0.00 -> 217.2 mm, vias 0 -> 5
- net N$38: track 213.5 -> 208.2 mm
- net N$37: track 208.6 -> 203.4 mm
- net N$33: track 205.3 -> 200.0 mm
- net N$31: track 194.2 -> 188.9 mm
- net N$34: track 200.3 -> 195.1 mm
- net N$32: track 188.9 -> 184.6 mm
- net N$36: track 219.8 -> 215.8 mm
- net N$9: track 0.00 -> 2.39 mm
- net N$27: track 0.00 -> 2.39 mm
- net N$26: track 0.00 -> 2.39 mm
- net N$25: track 0.00 -> 2.39 mm
- net N$24: track 0.00 -> 2.39 mm
- net N$12: track 0.00 -> 2.39 mm
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
Commit message: update silk
Parts:
- IC8, IC9: value 74HCT573N -> 74HCT574N
Other:
- board text added: "74HCT574N"
- board text removed: "74HCT573N"
Changed lines of the file:
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@@
 <text x="21.1328" y="-0.0635" size="0.0254" layer="22" font="vector" rot="MR0">C:/Users/aleksander.grodzki/Downloads/jabluszko.bmp</text>
 <text x="-22.8092" y="62.7507" size="1.27" layer="25" font="vector" ratio="15">Z80</text>
-<text x="-31.5214" y="32.4104" size="1.27" layer="25" font="vector" ratio="15">AT28C64</text>
-<text x="-30.5562" y="4.3434" size="1.27" layer="25" font="vector" ratio="15">6264</text>
+<text x="-31.2674" y="4.4704" size="1.27" layer="25" font="vector" ratio="15">AT28C64</text>
+<text x="-30.0482" y="32.5374" size="1.27" layer="25" font="vector" ratio="15">6264</text>
 <text x="-59.69" y="-5.08" size="1.27" layer="25" font="vector" ratio="15">HP35 clone
 (c)AG
@@
 <text x="-4.8514" y="88.2904" size="1.27" layer="25" font="vector" ratio="15">74HCT138N</text>
 <text x="-4.8514" y="111.1504" size="1.27" layer="25" font="vector" ratio="15">74HCT541N</text>
-<text x="-40.4114" y="132.7404" size="1.27" layer="25" font="vector" ratio="15">74HCT573N</text>
-<text x="-4.8514" y="132.7404" size="1.27" layer="25" font="vector" ratio="15">74HCT573N</text>
+<text x="-40.4114" y="132.7404" size="1.27" layer="25" font="vector" ratio="15">74HCT574N</text>
+<text x="-4.8514" y="132.7404" size="1.27" layer="25" font="vector" ratio="15">74HCT574N</text>
 <text x="30.7086" y="132.7404" size="1.27" layer="25" font="vector" ratio="15">74HCT154N</text>
 </plain>
@@
 <attribute name="VALUE" x="-7.493" y="88.265" size="1.27" layer="27" font="vector" ratio="15"/>
 </element>
-<element name="IC9" library="74xx-eu" package="DIL20" value="74HCT573N" x="-35.56" y="133.35" smashed="yes">
+<element name="IC9" library="74xx-eu" package="DIL20" value="74HCT574N" x="-35.56" y="133.35" smashed="yes">
 <attribute name="NAME" x="-48.641" y="130.302" size="1.27" layer="25" font="vector" ratio="15" rot="R90"/>
 <attribute name="VALUE" x="-45.339" y="132.969" size="1.27" layer="27" font="vector" ratio="15"/>
 </element>
-<element name="IC8" library="74xx-eu" package="DIL20" value="74HCT573N" x="0" y="133.35" smashed="yes">
+<element name="IC8" library="74xx-eu" package="DIL20" value="74HCT574N" x="0" y="133.35" smashed="yes">
 <attribute name="NAME" x="-13.081" y="130.302" size="1.27" layer="25" font="vector" ratio="15" rot="R90"/>
 <attribute name="VALUE" x="-9.779" y="132.969" size="1.27" layer="27" font="vector" ratio="15"/>
