File: hardware/HP35_Z80.sch (EAGLE design)
At the start: 82 parts, among them IC4 74HCT32N, IC5 74HCT154N, IC6 74HCT138N, IC7 74HCT541N, IC8 74HCT573N, IC9 74HCT573N, X1 MINI-USB-32005-301, X2 MINI-USB-32005-301

Commit message: add gerbers
Connections:
- new net CS: IC2G$1.!CE, IC4C.O
- net /MREQ: now also IC4C.I1
- net A15: now also IC4C.I0; no longer IC2G$1.!CE
- net GND: no longer IC4C.I0, IC4C.I1
Changed lines of the file:
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@@
 <label x="-208.28" y="-5.08" size="1.778" layer="95"/>
 <pinref part="IC1" gate="1" pin="A15"/>
-<wire x1="-200.66" y1="-5.08" x2="-200.66" y2="-2.54" width="0.1524" layer="91"/>
-<pinref part="IC2" gate="G$1" pin="!CE"/>
-<wire x1="-200.66" y1="-2.54" x2="-190.5" y2="-2.54" width="0.1524" layer="91"/>
+</segment>
+<segment>
+<pinref part="IC4" gate="C" pin="I0"/>
+<wire x1="-320.04" y1="-10.16" x2="-335.28" y2="-10.16" width="0.1524" layer="91"/>
+<label x="-330.2" y="-10.16" size="1.778" layer="95"/>
 </segment>
 <segment>
@@
 <wire x1="-320.04" y1="-38.1" x2="-325.12" y2="-38.1" width="0.1524" layer="91"/>
 <junction x="-325.12" y="-38.1"/>
-<wire x1="-325.12" y1="-33.02" x2="-325.12" y2="-15.24" width="0.1524" layer="91"/>
-<pinref part="IC4" gate="C" pin="I0"/>
-<wire x1="-325.12" y1="-15.24" x2="-325.12" y2="-10.16" width="0.1524" layer="91"/>
-<wire x1="-325.12" y1="-10.16" x2="-320.04" y2="-10.16" width="0.1524" layer="91"/>
-<pinref part="IC4" gate="C" pin="I1"/>
-<wire x1="-320.04" y1="-15.24" x2="-325.12" y2="-15.24" width="0.1524" layer="91"/>
-<junction x="-325.12" y="-15.24"/>
-<junction x="-325.12" y="-33.02"/>
 </segment>
 <segment>
@@
 <label x="-330.2" y="10.16" size="1.778" layer="95"/>
 </segment>
+<segment>
+<pinref part="IC4" gate="C" pin="I1"/>
+<wire x1="-320.04" y1="-15.24" x2="-335.28" y2="-15.24" width="0.1524" layer="91"/>
+<label x="-330.2" y="-15.24" size="1.778" layer="95"/>
+</segment>
 </net>
 <net name="/IORQ" class="0">
@@
 </segment>
 </net>
+<net name="CS" class="0">
+<segment>
+<pinref part="IC4" gate="C" pin="O"/>
+<wire x1="-294.64" y1="-12.7" x2="-281.94" y2="-12.7" width="0.1524" layer="91"/>
+<label x="-289.56" y="-12.7" size="1.778" layer="95"/>
+</segment>
+<segment>
+<pinref part="IC2" gate="G$1" pin="!CE"/>
+<wire x1="-190.5" y1="-2.54" x2="-198.12" y2="-2.54" width="0.1524" layer="91"/>
+<label x="-198.12" y="-2.54" size="1.778" layer="95"/>
+</segment>
+</net>

Commit message: update pcb
Parts:
- added R10, R11, R12, R13, R14, R15, R16, R17: (no value), rcl:R-EU_R1206
Connections:
- removed net N$35: DIS1.P$11, DIS2.P$11, DIS3.P$11, DIS4.P$11, IC9A.1Q
- new net N$10: IC9A.7Q, R16.1
- new net N$11: IC9A.6Q, R15.1
- new net N$12: IC9A.5Q, R14.1
- new net N$24: IC9A.4Q, R13.1
- new net N$25: IC9A.3Q, R12.1
- new net N$26: IC9A.2Q, R11.1
- new net N$27: IC9A.1Q, R10.1
- new net N$28: DIS1.P$11, DIS2.P$11, DIS3.P$11, DIS4.P$11, R10.2
- new net N$9: IC9A.8Q, R17.1
- net N$31: now also R17.2; no longer IC9A.8Q
- net N$32: now also R16.2; no longer IC9A.7Q
- net N$33: now also R15.2; no longer IC9A.6Q
- net N$34: now also R14.2; no longer IC9A.5Q
- net N$36: now also R11.2; no longer IC9A.2Q
- net N$37: now also R12.2; no longer IC9A.3Q
- net N$38: now also R13.2; no longer IC9A.4Q

Commit message: update silk
Parts:
- IC8, IC9: value 74HCT573N -> 74HCT574N
Changed lines of the file:
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@@
 <part name="P+20" library="supply1" deviceset="+5V" device=""/>
 <part name="IC6" library="74xx-eu" deviceset="74*138" device="N" technology="HCT"/>
-<part name="IC9" library="74xx-eu" deviceset="74*573" device="N" technology="HCT"/>
-<part name="IC8" library="74xx-eu" deviceset="74*573" device="N" technology="HCT"/>
+<part name="IC9" library="74xx-eu" deviceset="74*573" device="N" technology="HCT" value="74HCT574N"/>
+<part name="IC8" library="74xx-eu" deviceset="74*573" device="N" technology="HCT" value="74HCT574N"/>
 <part name="GND19" library="supply1" deviceset="GND" device=""/>
 <part name="IC7" library="74xx-eu" deviceset="74*541" device="N" technology="HCT"/>
